Commit message: kurang optimal setelah mapping dan mappingnya masih jelek

File: src/asv_description/urdf/asv_kki_2026.urdf.xacro (robot description, xacro)
@@ -287,5 +287,5 @@
   </link>
   <joint name="lidar_joint" type="fixed">
-    <origin xyz="0.036 0 0.520" rpy="0 0 0"/>
+    <origin xyz="0.036 0 0.150" rpy="0 0 0"/>
     <parent link="base_link"/>
     <child link="lidar_link"/>
